File: hardware/motion-carrier/conditioning.kicad_sch (KiCad schematic)
At the start: 4 parts

Commit message: fix(hardware): regenerate schematics, symbol library and PDFs
Regenerated output of the preceding fix-wave commits (contactor topology,
devkit pin order, field_gap/arrow-legibility fixes, 74LVC14 fields,
zero-length wire removal). ERC clean (0 violations on all three projects)
and check_pins reports 0 mismatches.

Co-Authored-By: Claude Opus 5 (1M context) <noreply@anthropic.com>
Claude-Session: https://claude.ai/code/session_01N1nWXzYgvFT6pqfHGhLK6P
Changed lines of the file:
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@@
 				(font
 					(size 1 1))
-				(justify right)))
+				(justify left)))
 		(property "Footprint" ""
 			(at 39.37 50.8 90)
