File: hardware/motion-carrier/motion-carrier.kicad_pcb (KiCad board)
At the start: 2 copper layers, 140 x 80 mm, 32 parts, among them J1 ESP32 devkit left row, J2 ESP32 devkit right row, J3 5V IN from buck, J4 TB6600 PUL+ PUL- DIR+ DIR- EN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, J5 RELAY +5V GND IN, J6 HOME GND TOP GND DRV_ALM GND, J7 PROBE GND FOOT GND STOP GND, J8 LINK to panel: GND TX RX

Commit message: fix(hardware): move the motion carrier link header away from the antenna
Co-Authored-By: Claude Opus 5 (1M context) <noreply@anthropic.com>
Claude-Session: https://claude.ai/code/session_01N1nWXzYgvFT6pqfHGhLK6P
Parts:
- moved J8 130.0 mm to (105.0, 136.0)
Routing:
- net /LINK_TX: track 28.1 -> 113.5 mm
- net /LINK_RX: track 26.2 -> 110.1 mm
- net /TOP_IN: track 100.5 -> 76.7 mm
- net +5V: track 133.8 -> 151.4 mm, vias 0 -> 1
- net /STEP: track 129.6 -> 146.9 mm
- net /DIR: track 134.3 -> 122.2 mm
- net /ENABLE: track 126.3 -> 120.6 mm
- net /HOME_IN: track 87.7 -> 84.6 mm
- net /PROBE_IN: track 56.1 -> 53.2 mm
- net /DRV_ALM_IN: track 72.1 -> 74.6 mm
- net /RELAY_IN: track 80.3 -> 78.4 mm
- net +3V3: track 197.9 -> 196.7 mm
- net GND: vias 53 -> 46

Commit message: fix(hardware): rectangular motion holes, shared link labels, regenerate boards
- motion carrier: M3 holes (4,4) (93,4) (4,56.5) (93,56.5), 89 x 52.5 mm, asserted
  as a rectangle, >=4 mm from edges, clear of courtyards/text, >=10 mm from the
  antenna keep-out; pitch silkscreen; DRV_ALM block lifted 7.5 mm; J2 refdes moved
  below its tail
- J8 and panel J3 labelled GND / LINK_TX / LINK_RX with a straight-through note;
  panel R1-R5 moved down 1 mm to make room
- stitch-avoid is builder state on both boards
- README: hole coordinates and pitch, Freerouting version override, what
  regeneration overwrites

Co-Authored-By: Claude Opus 5 (1M context) <noreply@anthropic.com>
Claude-Session: https://claude.ai/code/session_01N1nWXzYgvFT6pqfHGhLK6P
Parts:
- moved H4 43.4 mm to (193.0, 156.5)
- moved H2 8.00 mm to (193.0, 104.0)
- moved C5 7.50 mm to (196.6, 138.0)
- moved D5 7.50 mm to (192.6, 135.5)
- moved R10 7.50 mm to (196.6, 151.0)
- moved R9 7.50 mm to (192.6, 151.0)
- moved H3 5.50 mm to (104.0, 156.5)
Routing:
- net +5V: track 151.4 -> 133.1 mm, vias 1 -> 0
- net /DRV_ALM_FIELD: track 25.5 -> 33.0 mm
- net /DIR: track 122.2 -> 129.1 mm
- net /PROBE_IN: track 53.2 -> 59.9 mm
- net /TOP_IN: track 76.7 -> 70.1 mm, vias 1 -> 0
- net /DRV_ALM_IN: track 74.6 -> 68.1 mm
- net +3V3: track 196.7 -> 201.1 mm
- net /STEP: track 146.9 -> 149.1 mm
- net /RELAY_IN: track 78.4 -> 80.3 mm
- net /HOME_IN: track 84.6 -> 83.8 mm
- net GND: vias 46 -> 32
Other:
- board text added: "LINK: straight-through 1-1 2-2 3-3"
- board text added: "LINK_RX"
- board text added: "LINK_TX"
- board text added: "M3 HOLES 89 x 52.5 mm PITCH - VERIFY CLIPS"
- board text removed: "LINK"
- board text removed: "RX"
- board text removed: "TX"
