File: hardware/panel-carrier/panel-carrier.kicad_sch (KiCad schematic)
At the start: 16 parts, among them J1 display P3: IO6 IO7 IO15 IO16, J2 display P4: GND 3.3V IO17 IO18, J3 LINK to motion: GND TX RX, J4 MPG +5V GND A B, J5 5V IN from buck, J6 BUTTONS A0-A6, COM, J7 ROUTER LED + -, U1 74LVC14, U2 MCP23017 @0x20

Commit message: fix(hardware): regenerate schematics, symbol library and PDFs
Regenerated output of the preceding fix-wave commits (contactor topology,
devkit pin order, field_gap/arrow-legibility fixes, 74LVC14 fields,
zero-length wire removal). ERC clean (0 violations on all three projects)
and check_pins reports 0 mismatches.

Co-Authored-By: Claude Opus 5 (1M context) <noreply@anthropic.com>
Claude-Session: https://claude.ai/code/session_01N1nWXzYgvFT6pqfHGhLK6P
Changed lines of the file:
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@@
 				(hide yes)))
 		(property "Value" "GND"
-			(at 17.78 86.36 90)
+			(at 22.86 86.36 90)
 			(effects
 				(font
@@
 				(hide yes)))
 		(property "Value" "+3V3"
-			(at 17.78 88.9 90)
-			(effects
-				(font
-					(size 1 1))
-				(justify right)))
+			(at 22.86 88.9 90)
+			(effects
+				(font
+					(size 1 1))
+				(justify left)))
 		(property "Footprint" ""
 			(at 25.4 88.9 90)
@@
 				(hide yes)))
 		(property "Value" "+5V"
-			(at 17.78 162.56 90)
-			(effects
-				(font
-					(size 1 1))
-				(justify right)))
+			(at 22.86 162.56 90)
+			(effects
+				(font
+					(size 1 1))
+				(justify left)))
 		(property "Footprint" ""
 			(at 25.4 162.56 90)
@@
 				(hide yes)))
 		(property "Value" "GND"
-			(at 17.78 165.1 90)
+			(at 22.86 165.1 90)
 			(effects
 				(font
@@
 				(hide yes)))
 		(property "Value" "+5V"
-			(at 17.78 203.2 90)
-			(effects
-				(font
-					(size 1 1))
-				(justify right)))
+			(at 22.86 203.2 90)
+			(effects
+				(font
+					(size 1 1))
+				(justify left)))
 		(property "Footprint" ""
 			(at 25.4 203.2 90)
@@
 				(hide yes)))
 		(property "Value" "GND"
-			(at 17.78 205.74 90)
+			(at 22.86 205.74 90)
 			(effects
 				(font
@@
 				(justify left)
 				(hide yes)))
-		(property "Datasheet" ""
+		(property "Datasheet" "https://www.ti.com/lit/ds/symlink/sn74lvc14a.pdf"
+			(at 114.3 38.1 0)
+			(effects
+				(font
+					(size 1.27 1.27))
+				(justify left)
+				(hide yes)))
+		(property "Description" "Hex Schmitt-trigger inverter, 5 V tolerant inputs, 1.65-5.5 V"
 			(at 114.3 38.1 0)
 			(effects
@@
 				(justify left)
 				(hide yes)))
-		(property "Datasheet" ""
+		(property "Datasheet" "https://www.ti.com/lit/ds/symlink/sn74lvc14a.pdf"
+			(at 114.3 58.42 0)
+			(effects
+				(font
+					(size 1.27 1.27))
+				(justify left)
+				(hide yes)))
+		(property "Description" "Hex Schmitt-trigger inverter, 5 V tolerant inputs, 1.65-5.5 V"
 			(at 114.3 58.42 0)
 			(effects
@@
 				(justify left)
 				(hide yes)))
-		(property "Datasheet" ""
+		(property "Datasheet" "https://www.ti.com/lit/ds/symlink/sn74lvc14a.pdf"
+			(at 114.3 78.74 0)
+			(effects
+				(font
+					(size 1.27 1.27))
+				(justify left)
+				(hide yes)))
+		(property "Description" "Hex Schmitt-trigger inverter, 5 V tolerant inputs, 1.65-5.5 V"
 			(at 114.3 78.74 0)
 			(effects
@@
 				(justify left)
 				(hide yes)))
-		(property "Datasheet" ""
+		(property "Datasheet" "https://www.ti.com/lit/ds/symlink/sn74lvc14a.pdf"
+			(at 114.3 99.06 0)
+			(effects
+				(font
+					(size 1.27 1.27))
+				(justify left)
+				(hide yes)))
+		(property "Description" "Hex Schmitt-trigger inverter, 5 V tolerant inputs, 1.65-5.5 V"
 			(at 114.3 99.06 0)
 			(effects
@@
 				(justify left)
 				(hide yes)))
-		(property "Datasheet" ""
+		(property "Datasheet" "https://www.ti.com/lit/ds/symlink/sn74lvc14a.pdf"
+			(at 114.3 119.38 0)
+			(effects
+				(font
+					(size 1.27 1.27))
+				(justify left)
+				(hide yes)))
+		(property "Description" "Hex Schmitt-trigger inverter, 5 V tolerant inputs, 1.65-5.5 V"
 			(at 114.3 119.38 0)
 			(effects
@@
 				(justify left)
 				(hide yes)))
-		(property "Datasheet" ""
+		(property "Datasheet" "https://www.ti.com/lit/ds/symlink/sn74lvc14a.pdf"
+			(at 114.3 139.7 0)
+			(effects
+				(font
+					(size 1.27 1.27))
+				(justify left)
+				(hide yes)))
+		(property "Description" "Hex Schmitt-trigger inverter, 5 V tolerant inputs, 1.65-5.5 V"
 			(at 114.3 139.7 0)
 			(effects
@@
 				(justify left)
 				(hide yes)))
-		(property "Datasheet" ""
+		(property "Datasheet" "https://www.ti.com/lit/ds/symlink/sn74lvc14a.pdf"
+			(at 114.3 180.34 0)
+			(effects
+				(font
+					(size 1.27 1.27))
+				(justify left)
+				(hide yes)))
+		(property "Description" "Hex Schmitt-trigger inverter, 5 V tolerant inputs, 1.65-5.5 V"
 			(at 114.3 180.34 0)
 			(effects
@@
 				(hide yes)))
 		(property "Value" "GND"
-			(at 205.74 116.84 90)
+			(at 231.14 116.84 90)
 			(effects
 				(font
@@
 				(hide yes)))
 		(property "Value" "GND"
-			(at 205.74 119.38 90)
+			(at 231.14 119.38 90)
 			(effects
 				(font
@@
 				(hide yes)))
 		(property "Value" "GND"
-			(at 205.74 121.92 90)
+			(at 231.14 121.92 90)
 			(effects
 				(font
@@
 				(hide yes)))
 		(property "Value" "+3V3"
-			(at 205.74 104.14 90)
-			(effects
-				(font
-					(size 1 1))
-				(justify right)))
+			(at 231.14 104.14 90)
+			(effects
+				(font
+					(size 1 1))
+				(justify left)))
 		(property "Footprint" ""
 			(at 233.68 104.14 90)
@@
 				(hide yes)))
 		(property "Value" "GND"
-			(at 254 162.56 0)
+			(at 254 137.16 0)
 			(effects
 				(font
@@
 				(hide yes)))
 		(property "Value" "+3V3"
-			(at 254 40.64 0)
-			(effects
-				(font
+			(at 254 66.04 0)
+			(effects
+				(font
