File: hardware/system/low-voltage.kicad_sch (KiCad schematic)
At the start: 15 parts, among them M10 Buck 5 V >=2 A, M11 Motion carrier, M12 TB6600 1/8 step, M13 Stepper motor, M14 5 V relay module, M15 HOME bottom limit NC, M16 TOP limit NC, M17 Touch plate + clip on bit, M18 Foot pedal NO, M19 STOP flush NO, M20 Panel carrier, M21 Guition JC4827W543C, M22 MPG ZS80 100 PPR 5 V, M23 Panel buttons + rough/fine, M24 ROUTER LED

Commit message: fix(hardware): put the fuse before the E-stop and switch L and N at the contactor
Decided 2026-09-14: the mains order is RCD, fuse, E-stop, and the
router contactor is 2-pole so the router is isolated whichever way
round the supply is wired. The live net after the E-stop is renamed
L_ESTOP. BOM block A, WIRING-RevH diagrams 1 and 5 and the spec now
agree with the drawing; the key switch stays between the relay
contact and coil A1.

Co-Authored-By: Claude Opus 5 (1M context) <noreply@anthropic.com>
Claude-Session: https://claude.ai/code/session_01N1nWXzYgvFT6pqfHGhLK6P
Connections:
- net L_FUSED renamed L_ESTOP
Changed lines of the file:
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@@
 			(type default))
 )
-	(global_label "L_FUSED"
+	(global_label "L_ESTOP"
 		(shape bidirectional)
 		(at 314.96 124.46 0)
